Commit message: single arm track desired trajectory properly

File: urdf/single_6dof_arm.xacro (robot description, xacro)
@@ -116,5 +116,5 @@
       <mu1>0.9</mu1>
       <mu2>0.9</mu2>
-      <material>Gazebo/Grey</material>
+      <material>Gazebo/White</material>
       <self_collide>1</self_collide>
       <kp value="1000000.0"/>
@@ -124,4 +124,12 @@
       <mu1>0.9</mu1>
       <mu2>0.9</mu2>
+      <material>Gazebo/DarkGrey</material>
+      <self_collide>1</self_collide>
+      <kp value="1000000.0"/>
+      <kd value="1.0"/>
+  </gazebo>
+  <gazebo reference="arm_two">
+      <mu1>0.9</mu1>
+      <mu2>0.9</mu2>
       <material>Gazebo/White</material>
       <self_collide>1</self_collide>
@@ -129,24 +137,16 @@
       <kd value="1.0"/>
   </gazebo>
-  <gazebo reference="arm_two">
-      <mu1>0.9</mu1>
-      <mu2>0.9</mu2>
-      <material>Gazebo/Grey</material>
-      <self_collide>1</self_collide>
-      <kp value="1000000.0"/>
-      <kd value="1.0"/>
-  </gazebo>
   <gazebo reference="arm_three">
       <mu1>0.9</mu1>
       <mu2>0.9</mu2>
+      <material>Gazebo/DarkGrey</material>
+      <self_collide>1</self_collide>
+      <kp value="1000000.0"/>
+      <kd value="1.0"/>
+  </gazebo>
+  <gazebo reference="arm_four">
+      <mu1>0.9</mu1>
+      <mu2>0.9</mu2>
       <material>Gazebo/White</material>
-      <self_collide>1</self_collide>
-      <kp value="1000000.0"/>
-      <kd value="1.0"/>
-  </gazebo>
-  <gazebo reference="arm_four">
-      <mu1>0.9</mu1>
-      <mu2>0.9</mu2>
-      <material>Gazebo/Grey</material>
       <self_collide>1</self_collide>
       <kp value="1000000.0"/>

Commit message: complete inverse dynamics algorithm applied to the single-arm robot

File: urdf/single_6dof_arm.xacro (robot description, xacro)
@@ -341,5 +341,5 @@
   </link>
   <joint name="arm_three_to_arm_two" type="revolute">
-    <axis xyz="0 0 1"/>
+    <axis xyz="1 0 0"/>
     <limit effort="50" lower="-3.14" upper="3.14" velocity="4"/>
     <origin rpy="0 0 0" xyz="${length_arm_two} 0 0"/>

Commit message: box added to xacro model

File: urdf/single_6dof_arm.xacro (robot description, xacro)
@@ -161,4 +161,12 @@
       <kd value="1.0"/>
   </gazebo>
+  <gazebo reference="box">
+      <mu1>0.9</mu1>
+      <mu2>0.9</mu2>
+      <material>Gazebo/Green</material>
+      <self_collide>1</self_collide>
+      <kp value="1000000.0"/>
+      <kd value="1.0"/>
+  </gazebo>
   <link name="world"/>
   <joint name="trunk_to_world" type="fixed">
@@ -433,5 +441,5 @@
     </inertial>
   </link>
-  <!-- <joint name="box_to_hand" type="fixed">
+  <joint name="box_to_hand" type="fixed">
       <origin rpy="0 0 0" xyz="0 ${width_box/2 + width_arm/2} 0"/>
       <parent link="hand"/>
@@ -460,5 +468,5 @@
         	  izz="${i_box_zz}"/>
       </inertial>
-  </link> -->
+  </link>
   <transmission name="tran1">
     <type>transmission_interface/SimpleTransmission</type>

Commit message: arm does not follow trajectory properly

File: urdf/single_6dof_arm.xacro (robot description, xacro)
@@ -48,7 +48,7 @@
   <xacro:property name="friction_ratio_arm_three" value="1" />
   <xacro:property name="damping_ratio_arm_four" value="1" />
-  <xacro:property name="friction_ratio_arm_four" value="1" />
+  <xacro:property name="friction_ratio_arm_four" value=".1" />
   <xacro:property name="damping_ratio_hand" value="1" />
-  <xacro:property name="friction_ratio_hand" value="1" />
+  <xacro:property name="friction_ratio_hand" value=".1" />
   <xacro:property name="i_trunk_xx" value="0.011253" />
   <xacro:property name="i_trunk_yy" value="0.036203" />

Commit message: commit before initializing an issue

File: urdf/single_6dof_arm.xacro (robot description, xacro)
@@ -40,5 +40,5 @@
   <xacro:property name="height_box" value="0.15" />
   <xacro:property name="damping_ratio_arm_zero" value="1" />
-  <xacro:property name="friction_ratio_arm_zero" value=".1" />
+  <xacro:property name="friction_ratio_arm_zero" value="1" />
   <xacro:property name="damping_ratio_arm_one" value="1" />
   <xacro:property name="friction_ratio_arm_one" value="1" />

Commit message: trunk removed

File: urdf/single_6dof_arm.xacro (robot description, xacro)
@@ -19,5 +19,5 @@
   <xacro:property name="mass_arm_four" value=".5" />
   <xacro:property name="mass_hand" value="1" />
-  <xacro:property name="mass_box" value=".1" />
+  <xacro:property name="mass_box" value=".01" />
   <xacro:property name="width_trunk" value="0.2" />
   <xacro:property name="length_trunk" value="0.3" />
@@ -81,13 +81,8 @@
   <xacro:property name="i_box_yy" value="${mass_box/12*(width_box*width_box + height_box*height_box)}" />
   <xacro:property name="i_box_zz" value="${mass_box/12*(width_box*width_box + length_box*length_box)}" />
-  <gazebo reference="trunk">
-      <mu1>0.9</mu1>
-      <mu2>0.9</mu2>
-      <material>Gazebo/White</material>
-  </gazebo>
   <gazebo reference="world">
       <static>true</static>
   </gazebo>
-  <gazebo reference="trunk">
+  <gazebo reference="child_neck">
       <mu1>0.9</mu1>
       <mu2>0.9</mu2>
@@ -97,5 +92,13 @@
       <kd value="1.0"/>
   </gazebo>
-  <gazebo reference="parent_neck">
+  <gazebo reference="arm_zero">
+      <mu1>0.9</mu1>
+      <mu2>0.9</mu2>
+      <material>Gazebo/White</material>
+      <self_collide>1</self_collide>
+      <kp value="1000000.0"/>
+      <kd value="1.0"/>
+  </gazebo>
+  <gazebo reference="arm_one">
       <mu1>0.9</mu1>
       <mu2>0.9</mu2>
@@ -105,5 +108,13 @@
       <kd value="1.0"/>
   </gazebo>
-  <gazebo reference="child_neck">
+  <gazebo reference="arm_two">
+      <mu1>0.9</mu1>
+      <mu2>0.9</mu2>
+      <material>Gazebo/White</material>
+      <self_collide>1</self_collide>
+      <kp value="1000000.0"/>
+      <kd value="1.0"/>
+  </gazebo>
+  <gazebo reference="arm_three">
       <mu1>0.9</mu1>
       <mu2>0.9</mu2>
@@ -113,5 +124,5 @@
       <kd value="1.0"/>
   </gazebo>
-  <gazebo reference="arm_zero">
+  <gazebo reference="arm_four">
       <mu1>0.9</mu1>
       <mu2>0.9</mu2>
@@ -121,36 +132,4 @@
       <kd value="1.0"/>
   </gazebo>
-  <gazebo reference="arm_one">
-      <mu1>0.9</mu1>
-      <mu2>0.9</mu2>
-      <material>Gazebo/DarkGrey</material>
-      <self_collide>1</self_collide>
-      <kp value="1000000.0"/>
-      <kd value="1.0"/>
-  </gazebo>
-  <gazebo reference="arm_two">
-      <mu1>0.9</mu1>
-      <mu2>0.9</mu2>
-      <material>Gazebo/White</material>
-      <self_collide>1</self_collide>
-      <kp value="1000000.0"/>
-      <kd value="1.0"/>
-  </gazebo>
-  <gazebo reference="arm_three">
-      <mu1>0.9</mu1>
-      <mu2>0.9</mu2>
-      <material>Gazebo/DarkGrey</material>
-      <self_collide>1</self_collide>
-      <kp value="1000000.0"/>
-      <kd value="1.0"/>
-  </gazebo>
-  <gazebo reference="arm_four">
-      <mu1>0.9</mu1>
-      <mu2>0.9</mu2>
-      <material>Gazebo/White</material>
-      <self_collide>1</self_collide>
-      <kp value="1000000.0"/>
-      <kd value="1.0"/>
-  </gazebo>
   <gazebo reference="hand">
       <mu1>0.9</mu1>
@@ -170,64 +149,7 @@
   </gazebo>
   <link name="world"/>
-  <joint name="trunk_to_world" type="fixed">
-    <origin rpy="0 0 0" xyz="0 0 0"/>
-    <parent link="world"/>
-    <child link="trunk"/>
-  </joint>
-  <!-- Base Link -->
-  <link name="trunk">
-    <collision>
-      <origin rpy="0 0 0" xyz="0 0 0"/>
-      <geometry>
-	       <box size="${width_trunk} ${length_trunk} ${height_trunk}"/>
-      </geometry>
-    </collision>
-    <visual>
-      <origin rpy="0 0 0" xyz="0 0 0"/>
-      <geometry>
-	       <box size="${width_trunk} ${length_trunk} ${height_trunk}"/>
-      </geometry>
-      <material name="white"/>
-    </visual>
-    <inertial>
-      <origin rpy="0 0 0" xyz="0 0 0"/>
-      <mass value="${mass_trunk}"/>
-      <inertia
-        ixx="${i_trunk_xx}" ixy="0.0" ixz="0.0"
-    	  iyy="${i_trunk_yy}" iyz="0.0"
-    	  izz="${i_trunk_zz}"/>
-    </inertial>
-  </link>
-  <joint name="parent_neck_to_trunk" type="fixed">
-    <origin rpy="0 0 0" xyz="0 0.08 ${height_trunk/2}"/>
-    <parent link="trunk"/>
-    <child link="parent_neck"/>
-  </joint>
-  <link name="parent_neck">
-    <collision>
-      <origin rpy="0 0 0" xyz="0 0 ${height_parent_neck/2}"/>
-      <geometry>
-	       <box size="${width_parent_neck} ${length_parent_neck} ${height_parent_neck}"/>
-      </geometry>
-    </collision>
-    <visual>
-      <origin rpy="0 0 0" xyz="0 0 ${height_parent_neck/2}"/>
-      <geometry>
-	       <box size="${width_parent_neck} ${length_parent_neck} ${height_parent_neck}"/>
-      </geometry>
-      <material name="white"/>
-    </visual>
-    <inertial>
-      <origin rpy="0 0 0" xyz="0 0 ${height_parent_neck/2}"/>
-      <mass value="${mass_parent_neck}"/>
-      <inertia
-        ixx="${i_parent_neck_xx}" ixy="0.0" ixz="0.0"
-    	  iyy="${i_parent_neck_yy}" iyz="0.0"
-    	  izz="${i_parent_neck_zz}"/>
-    </inertial>
-  </link>
   <joint name="child_neck_to_parent_neck" type="fixed">
     <origin rpy="0 0 0" xyz="0 0 ${height_parent_neck}"/>
-    <parent link="parent_neck"/>
+    <parent link="world"/>
     <child link="child_neck"/>
   </joint>

Commit message: separate gain of acceleration for joints

File: urdf/single_6dof_arm.xacro (robot description, xacro)
@@ -18,6 +18,6 @@
   <xacro:property name="mass_arm_three" value=".5" />
   <xacro:property name="mass_arm_four" value=".5" />
-  <xacro:property name="mass_hand" value="1" />
-  <xacro:property name="mass_box" value=".01" />
+  <xacro:property name="mass_hand" value=".1" />
+  <xacro:property name="mass_box" value="1" />
   <xacro:property name="width_trunk" value="0.2" />
   <xacro:property name="length_trunk" value="0.3" />
@@ -46,5 +46,5 @@
   <xacro:property name="friction_ratio_arm_two" value="1" />
   <xacro:property name="damping_ratio_arm_three" value="1" />
-  <xacro:property name="friction_ratio_arm_three" value="1" />
+  <xacro:property name="friction_ratio_arm_three" value="5" />
   <xacro:property name="damping_ratio_arm_four" value="1" />
   <xacro:property name="friction_ratio_arm_four" value=".1" />
@@ -179,5 +179,5 @@
   <joint name="arm_zero_to_child_neck" type="revolute">
     <axis xyz="1 0 0"/>
-    <limit effort="50" lower="-3.14" upper="3.14" velocity="4"/>
+    <limit effort="50" lower="-6.28" upper="6.28" velocity="4"/>
     <origin rpy="0 0 0" xyz="${width_child_neck/2} 0 ${height_child_neck/2}"/>
     <parent link="child_neck"/>
@@ -210,5 +210,5 @@
   <joint name="arm_one_to_arm_zero" type="revolute">
     <axis xyz="0 0 1"/>
-    <limit effort="50" lower="-3.14" upper="3.14" velocity="4"/>
+    <limit effort="50" lower="-6.28" upper="6.28" velocity="4"/>
     <origin rpy="0 0 ${PI/3}" xyz="${width_arm} 0 0"/>  <!-- in parent link frame -->
     <parent link="arm_zero"/>
@@ -241,5 +241,5 @@
   <joint name="arm_two_to_arm_one" type="revolute">
     <axis xyz="0 0 1"/>
-    <limit effort="50" lower="-3.14" upper="3.14" velocity="4"/>
+    <limit effort="50" lower="-6.28" upper="6.28" velocity="4"/>
     <origin rpy="0 0 ${PI/3}" xyz="${length_arm_one} 0 0"/>
     <parent link="arm_one"/>
@@ -272,5 +272,5 @@
   <joint name="arm_three_to_arm_two" type="revolute">
     <axis xyz="1 0 0"/>
-    <limit effort="50" lower="-3.14" upper="3.14" velocity="4"/>
+    <limit effort="50" lower="-6.28" upper="6.28" velocity="4"/>
     <origin rpy="0 0 0" xyz="${length_arm_two} 0 0"/>
     <parent link="arm_two"/>
@@ -303,5 +303,5 @@
   <joint name="arm_four_to_arm_three" type="revolute">
     <axis xyz="0 0 1"/>
-    <limit effort="50" lower="-3.14" upper="3.14" velocity="4"/>
+    <limit effort="50" lower="-6.28" upper="6.28" velocity="4"/>
     <origin rpy="0 0 0" xyz="${length_arm_three} 0 0"/>
     <parent link="arm_three"/>
@@ -334,5 +334,5 @@
   <joint name="hand_to_arm_four" type="revolute">
     <axis xyz="0 0 1"/>
-    <limit effort="50" lower="-3.14" upper="3.14" velocity="4"/>
+    <limit effort="50" lower="-6.28" upper="6.28" velocity="4"/>
     <origin rpy="0 0 ${-PI/6}" xyz="${length_arm_four} 0 0"/>
     <parent link="arm_four"/>

Commit message: first result for trajectory generation.

File: urdf/single_6dof_arm.xacro (robot description, xacro)
@@ -18,5 +18,5 @@
   <xacro:property name="mass_arm_three" value=".5" />
   <xacro:property name="mass_arm_four" value=".5" />
-  <xacro:property name="mass_hand" value=".1" />
+  <xacro:property name="mass_hand" value="1" />
   <xacro:property name="mass_box" value="1" />
   <xacro:property name="width_trunk" value="0.2" />
@@ -46,7 +46,7 @@
   <xacro:property name="friction_ratio_arm_two" value="1" />
   <xacro:property name="damping_ratio_arm_three" value="1" />
-  <xacro:property name="friction_ratio_arm_three" value="5" />
+  <xacro:property name="friction_ratio_arm_three" value="1" />
   <xacro:property name="damping_ratio_arm_four" value="1" />
-  <xacro:property name="friction_ratio_arm_four" value=".1" />
+  <xacro:property name="friction_ratio_arm_four" value="1" />
   <xacro:property name="damping_ratio_hand" value="1" />
   <xacro:property name="friction_ratio_hand" value=".1" />
@@ -363,5 +363,5 @@
     </inertial>
   </link>
-  <joint name="box_to_hand" type="fixed">
+  <!-- <joint name="box_to_hand" type="fixed">
       <origin rpy="0 0 0" xyz="0 ${width_box/2 + width_arm/2} 0"/>
       <parent link="hand"/>
@@ -390,5 +390,5 @@
         	  izz="${i_box_zz}"/>
       </inertial>
-  </link>
+  </link> -->
   <transmission name="tran1">
     <type>transmission_interface/SimpleTransmission</type>

Commit message: seemingly, orientation tracking is working, by precise setting of friction

File: urdf/single_6dof_arm.xacro (robot description, xacro)
@@ -46,5 +46,5 @@
   <xacro:property name="friction_ratio_arm_two" value="1" />
   <xacro:property name="damping_ratio_arm_three" value="1" />
-  <xacro:property name="friction_ratio_arm_three" value="1" />
+  <xacro:property name="friction_ratio_arm_three" value="5" />
   <xacro:property name="damping_ratio_arm_four" value="1" />
   <xacro:property name="friction_ratio_arm_four" value="1" />
@@ -334,5 +334,5 @@
   <joint name="hand_to_arm_four" type="revolute">
     <axis xyz="0 0 1"/>
-    <limit effort="50" lower="-6.28" upper="6.28" velocity="4"/>
+    <limit effort="100" lower="-6.28" upper="6.28" velocity="10"/>
     <origin rpy="0 0 ${-PI/6}" xyz="${length_arm_four} 0 0"/>
     <parent link="arm_four"/>

Commit message: modification

File: urdf/single_6dof_arm.xacro (robot description, xacro)
@@ -46,5 +46,5 @@
   <xacro:property name="friction_ratio_arm_two" value="1" />
   <xacro:property name="damping_ratio_arm_three" value="1" />
-  <xacro:property name="friction_ratio_arm_three" value="5" />
+  <xacro:property name="friction_ratio_arm_three" value="10" />
   <xacro:property name="damping_ratio_arm_four" value="1" />
   <xacro:property name="friction_ratio_arm_four" value="1" />
